Commit message: working launch files

File: ros_ws/src/six_dof_arm_description/urdf/six_dof_arm.urdf (robot description, URDF)
Before this commit: robot six_dof_arm, 7 links, 6 joints
Links:
- removed link k0
- removed link k1
- removed link k2
- removed link k3
- removed link k4
- removed link k5
- added link link_0; collision box size=0.02 0.24 0.14; collision box size=0.16 0.10 0.1
- added link link_1; collision box size=0.02 0.3 0.14; collision cylinder length=0.06 radius=0.09
- added link link_2; collision cylinder length=0.10 radius=0.09; collision cylinder length=0.13 radius=0.07
- added link link_3; collision box size=0.12 0.20 0.12; visual mesh filename=package://six_dof_arm_description/meshes/link04.dae
- added link link_4; collision box size=0.14 0.02 0.12; collision cylinder length=0.026 radius=0.070
- added link link_5; collision cylinder length=0.02 radius=0.05; visual mesh filename=package://six_dof_arm_description/meshes/end_effector.dae
Joints:
- removed joint j0
- removed joint j1
- removed joint j2
- removed joint j3
- removed joint j4
- removed joint j5
- added joint joint_0: type revolute, parent base_link, child link_0, origin xyz=0.000 0.000 0.000 rpy=0.00 0.00 0.00, axis 0 0 1, limit lower=-3.14 upper=3.14 effort=80.0 velocity=2.01
- added joint joint_1: type revolute, parent link_0, child link_1, origin xyz=0.092 -0.160 0.120 rpy=0.00 0.00 0.00, axis 1 0 0, limit lower=0.0 upper=3.14 effort=50.0 velocity=2.01
- added joint joint_2: type revolute, parent link_1, child link_2, origin xyz=0.000 0.300 0.000 rpy=0.00 0.00 0.00, axis -1 0 0, limit lower=0.0872664626 upper=3.141592 effort=50.0 velocity=2.01
- added joint joint_3: type revolute, parent link_2, child link_3, origin xyz=-0.092 -0.080 0.104 rpy=0.00 0.00 0.00, axis 0 1 0, limit lower=-3.14 upper=3.14 effort=30.0 velocity=2.01
- added joint joint_4: type revolute, parent link_3, child link_4, origin xyz=0.00 -0.202 0.00 rpy=0.00 0.00 0.00, axis 1 0 0, limit lower=-1.57 upper=1.57 effort=10.0 velocity=2.01
- added joint joint_5: type revolute, parent link_4, child link_5, origin xyz=0.00 -0.062 0.00 rpy=0.00 0.00 0.00, axis 0 1 0, limit lower=-3.14 upper=3.14 effort=10.0 velocity=2.01

Commit message: working version

File: ros_ws/src/six_dof_arm_description/urdf/six_dof_arm.urdf (robot description, URDF)
Before this commit: robot six_dof_arm, 7 links, 6 joints
Joints:
- joint joint_4: axis 1 0 0 -> -1 0 0
